Commit message: Обновил структуру, потихоньку разбираюсь в ros2_control

File: urdf/base.xacro (robot description, xacro)
@@ -1,6 +1,8 @@
 <?xml version="1.0"?>
 <robot xmlns:xacro="http://www.ros.org/wiki/xacro">
+  <xacro:include filename="$(find delta_robot_ros2)/urdf/common_macro.xacro"/>
   <xacro:macro name="base" params="id base_radius base_height base_material_rgba">
     <link name="GSC">
+      <xacro:inertial_cylinder mass="0.1" length="${1}" radius="${1}"/>
     </link>
     <!-- Чтобы перевернуть систему исменить rpy (${pi} 0 0) -->
@@ -19,4 +21,5 @@
         </material>
       </visual>
+      <xacro:inertial_cylinder mass="1" length="${base_height}" radius="${base_radius}"/>
     </link>
   </xacro:macro>

File: urdf/delta_robot.xacro (robot description, xacro)
@@ -6,12 +6,13 @@
   <xacro:include filename="$(find delta_robot_ros2)/urdf/leg.xacro"/>
   <xacro:include filename="$(find delta_robot_ros2)/urdf/platform.xacro"/>
+  <xacro:include filename="$(find delta_robot_ros2)/urdf/robot_control.xacro"/>
 <!-- *********************************************************************** -->
   <!-- Параметры для основания и платформы -->
   <xacro:property name="base_radius" value="0.5"/>
-  <xacro:property name="base_height" value="0.1"/>
-  <xacro:property name="base_material_rgba" value="0.5 0.5 0.5 1"/>
+  <xacro:property name="base_height" value="0.05"/>
+  <xacro:property name="base_material_rgba" value="1 0 0 0.8"/>
   <xacro:property name="platform_radius" value="0.3"/>
-  <xacro:property name="platform_height" value="0.1"/>
-  <xacro:property name="platform_material_rgba" value="0.7 0.7 0.7 1"/>
+  <xacro:property name="platform_height" value="0.05"/>
+  <xacro:property name="platform_material_rgba" value="0 1 0 0.8"/>
   <xacro:property name="platform_initial_height" value="0.6"/>
 <!-- *********************************************************************** -->
@@ -37,3 +38,4 @@
   <xacro:leg prefix="leg_3" origin_xyz="${leg_3_origin_xyz}" origin_rpy="${leg_3_origin_rpy}"/>
 <!-- *********************************************************************** -->
+  <xacro:daleta_robot_control/>
 </robot>

File: urdf/leg.xacro (robot description, xacro)
@@ -1,4 +1,5 @@
 <?xml version="1.0"?>
 <robot xmlns:xacro="http://www.ros.org/wiki/xacro">
+  <xacro:include filename="$(find delta_robot_ros2)/urdf/common_macro.xacro"/>
 <!-- *********************************************************************** -->
   <!-- Simple transmission -->
@@ -25,4 +26,21 @@
     </joint>
     <xacro:simple_transmission joint_name="${prefix}_joint_1"/>
+    <!-- <ros2_control name="${prefix}_control" type="actuator">
+      <hardware>
+        <plugin>ros2_control_demo_hardware/GenericActuator</plugin>
+      </hardware>
+      <joint_state_broadcaster>
+        <plugin>joint_state_broadcaster/JointStateBroadcaster</plugin>
+        <joint>
+          <name>${prefix}_joint_1</name>
+        </joint>
+      </joint_state_broadcaster>
+      <controller>
+        <plugin>position_controllers/JointPositionController</plugin>
+        <joint>
+          <name>${prefix}_joint_1</name>
+        </joint>
+      </controller>
+    </ros2_control> -->
 <!-- *********************************************************************** -->
     <!-- Первое звено -->
@@ -36,4 +54,5 @@
         </material>
       </visual>
+      <xacro:inertial_cylinder mass="1" length="${0.4}" radius="${0.05}"/>
     </link>
 <!-- *********************************************************************** -->

File: urdf/platform.xacro (robot description, xacro)
@@ -1,4 +1,5 @@
 <?xml version="1.0"?>
 <robot xmlns:xacro="http://ros.org/wiki/xacro">
+  <xacro:include filename="$(find delta_robot_ros2)/urdf/common_macro.xacro"/>
   <xacro:macro name="platform" params="id platform_radius platform_height platform_material_rgba parent origin_xyz origin_rpy">
     <link name="${id}">
@@ -11,4 +12,5 @@
         </material>
       </visual>
+      <xacro:inertial_cylinder mass="1" length="${platform_height}" radius="${platform_radius}"/>
     </link>
     <!-- Шарнир соединяющий платформу с базой (возможно условно, если требуется для структуры URDF) -->
