Commit message: Насчтроил приметивное управление

File: urdf/delta_robot.xacro (robot description, xacro)
@@ -18,5 +18,5 @@
 <!-- *********************************************************************** -->
   <!-- Блок расчёта расположения и ориентации ног дельтаробота -->
-  <xacro:property name="base_offset_z" value="0.2"/>
+  <xacro:property name="base_offset_z" value="0"/>
   <xacro:property name="angle_deg_1" value="0"/>
   <xacro:property name="angle_deg_2" value="120"/>

File: urdf/leg.xacro (robot description, xacro)
@@ -23,13 +23,15 @@
       <child link="${prefix}_link_1"/>
       <axis xyz="0 1 0"/>
-      <limit lower="-${pi / 2}" upper="${pi / 2}" effort="1000" velocity="3"/>
+      <limit lower="-${pi / 3}" upper="${pi / 3}" effort="1000" velocity="3"/>
     </joint>
     <xacro:simple_transmission joint_name="${prefix}_joint_1"/>
 <!-- *********************************************************************** -->
+    <xacro:property name="leg_length" value="0.4"/>
     <!-- Первое звено -->
     <link name="${prefix}_link_1">
       <visual>
+        <origin xyz="0 0 ${leg_length / 2}"/>
         <geometry>
-          <cylinder length="0.4" radius="0.05"/>
+          <cylinder length="${leg_length}" radius="0.05"/>
         </geometry>
          <material name="material_link_1">

File: urdf/robot_control.xacro (robot description, xacro)
@@ -16,6 +16,6 @@
         <joint name="leg_1_joint_1">
             <command_interface name="position">
-                <param name="min">-1</param>
-                <param name="max">1</param>
+                <param name="min">- ${pi / 3}</param>
+                <param name="max">${pi / 3}</param>
             </command_interface>
             <state_interface name="position"/>
@@ -23,6 +23,6 @@
         <joint name="leg_2_joint_1">
             <command_interface name="position">
-                <param name="min">-1</param>
-                <param name="max">1</param>
+                <param name="min">- ${pi / 3}</param>
+                <param name="max">${pi / 3}</param>
             </command_interface>
             <state_interface name="position"/>
@@ -30,6 +30,6 @@
         <joint name="leg_3_joint_1">
             <command_interface name="position">
-                <param name="min">-1</param>
-                <param name="max">1</param>
+                <param name="min">- ${pi / 3}</param>
+                <param name="max">${pi / 3}</param>
             </command_interface>
             <state_interface name="position"/>
